File: f1-led-circuit-kicad/rgb_led_track_chain.kicad_sch (KiCad schematic)
At the start: 30 parts, among them U10 HD108-2020, U11 HD108-2020, U12 HD108-2020, U13 HD108-2020, U14 HD108-2020, U15 HD108-2020, U16 HD108-2020, U17 HD108-2020, U18 HD108-2020, U19 HD108-2020, U20 HD108-2020, U21 HD108-2020, U22 HD108-2020, U23 HD108-2020, U24 HD108-2020, U25 HD108-2020, U26 HD108-2020, U27 HD108-2020, U28 HD108-2020, U29 HD108-2020, U30 HD108-2020, U31 HD108-2020, U32 HD108-2020, U33 HD108-2020, U4 HD108-2020, U5 HD108-2020, U6 HD108-2020, U7 HD108-2020, U8 HD108-2020, U9 HD108-2020

Commit message: KiCad - Update RGB LED Chains - 124 LEDS represented
Parts:
- renumbered U5 to U34, U14 to U35, U23 to U36, U32 to U37, U4 to U38, U15 to U39, U24 to U40, U33 to U41, U6 to U42, U16 to U43, U25 to U44, U7 to U45, U17 to U46, U26 to U47, U8 to U48, U18 to U49, U27 to U50, U9 to U51, U19 to U52, U28 to U53, U10 to U54, U20 to U55, U29 to U56, U11 to U57, U21 to U58, U30 to U59, U12 to U60, U22 to U61, U31 to U62, U13 to U63
Connections:
- net CLOCK_CHAIN_4_TO_5 renamed DCKO
- net DATA_CHAIN_4_TO_5 renamed DOUT
- net MCU_CLOCK_1 renamed DCKI
- net MCU_DATA_1 renamed DIN
