File: kicad/f1-led-circuit.kicad_sch (KiCad schematic)
At the start: 38 parts, among them J1 USB_C_Receptacle_USB2.0_14P, J2 Conn_ARM_JTAG_SWD_10_F1, Q1 TSM085P03CV_RGG, SW1 SW_SPST, SW2 SW_SPST, SW3 SW_SPDT, U1 HD108-2020, U2 HD108-2020, U200 ESP32-C3-MINI-1, U201 MCP9701AT-E/TT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

Commit message: Update temperature sensor part number
Parts:
- U201: value MCP9701AT-E/TT -> MCP9701AT-E/LT; MPN MCP9701AT-E/TT -> MCP9701AT-E/LT
Changed lines of the file:
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@@
 			)
 		)
-		(property "Value" "MCP9701AT-E/TT"
+		(property "Value" "MCP9701AT-E/LT"
 			(at 357.886 26.924 0)
 			(effects
@@
 			)
 		)
-		(property "MPN" "MCP9701AT-E/TT"
+		(property "MPN" "MCP9701AT-E/LT"
 			(at 337.82 35.56 0)
 			(effects
