File: kicad/zandvoort_10x10/f1-led-circuit-10x10.kicad_pcb (KiCad board)
At the start: 2 copper layers, 100 x 100 mm, 142 parts, among them J1 USB_C_Receptacle_USB2.0_14P, J2 Conn_ARM_JTAG_SWD_10_F1, Q1 TSM085P03CV_RGG, SW1 SW_SPST, SW2 SW_SPST, SW3 SW_SPDT, U1 HD108-2020, U10 HD108-2020, U11 HD108-2020, U12 HD108-2020, U13 HD108-2020, U14 HD108-2020, U15 HD108-2020, U16 HD108-2020, U17 HD108-2020, U18 HD108-2020, U19 HD108-2020, U2 HD108-2020, U20 HD108-2020, U200 ESP32-C3-MINI-1, U201 MCP9701AT-E/TT, U202 LDLN050, U203 NUF2042XV6T1G, U21 HD108-2020, U22 HD108-2020, U23 HD108-2020, U24 HD108-2020, U25 HD108-2020, U26 HD108-2020, U27 HD108-2020, U28 HD108-2020, U29 HD108-2020, U3 HD108-2020, U30 HD108-2020, U31 HD108-2020, U32 HD108-2020, U33 HD108-2020, U34 HD108-2020, U35 HD108-2020, U36 HD108-2020, U37 HD108-2020, U38 HD108-2020, U39 HD108-2020, U4 HD108-2020, U40 HD108-2020, U41 HD108-2020, U42 HD108-2020, U43 HD108-2020, U44 HD108-2020, U45 HD108-2020, U46 HD108-2020, U47 HD108-2020, U48 HD108-2020, U49 HD108-2020, U5 HD108-2020, U50 HD108-2020, U51 HD108-2020, U52 HD108-2020, U53 HD108-2020, U54 HD108-2020, U55 HD108-2020, U56 HD108-2020, U57 HD108-2020, U58 HD108-2020, U59 HD108-2020, U6 HD108-2020, U60 HD108-2020, U61 HD108-2020, U62 HD108-2020, U63 HD108-2020, U64 HD108-2020, U65 HD108-2020, U66 HD108-2020, U67 HD108-2020, U68 HD108-2020, U69 HD108-2020, U7 HD108-2020, U70 HD108-2020, U71 HD108-2020, U72 HD108-2020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

Commit message: Create seaparate 20x20 and 10x10 Kicad projects in kicad root
Changed lines of the file:
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@@
 		)
 		(pad "3" smd rect
-			(at -0.7 0.800001 19)
+			(at -0.7 0.800002 19)
 			(size 0.6 0.4)
 			(layers "F.Cu" "F.Paste" "F.Mask")
@@
 		)
 		(pad "4" smd rect
-			(at 0.7 -0.800001 19)
+			(at 0.7 -0.800002 19)
 			(size 0.6 0.4)
 			(layers "F.Cu" "F.Paste" "F.Mask")
