File: kicad/zandvoort_10x10/f1-led-circuit-10x10.kicad_sch (KiCad schematic)
At the start: 38 parts, among them J1 USB_C_Receptacle_USB2.0_14P, J2 Conn_ARM_JTAG_SWD_10_F1, Q1 TSM085P03CV_RGG, SW1 SW_SPST, SW2 SW_SPST, SW3 SW_SPDT, U1 HD108-2020, U2 HD108-2020, U200 ESP32-C3-MINI-1, U201 MCP9701AT-E/LT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

Commit message: Create seaparate 20x20 and 10x10 Kicad projects in kicad root
Connections:
- net GND: now also U202.GND (4); no longer U202.4 (GND), U202.9 (GND)
- net LED_CHAIN1/DCKI: now also U6.3 (DCKO); no longer U6.2 (DCKO)
- net LED_CHAIN1/DIN: now also U6.2 (DOUT); no longer U6.3 (DOUT)
- net at U4.2 (DOUT): now also U5.6 (DIN); no longer U5.5 (DCKI)
- net at U4.3 (DCKO): now also U5.5 (DCKI); no longer U5.6 (DIN)
- net at U4.5 (DCKI): now also U3.3 (DCKO); no longer U3.2 (DCKO)
- net at U4.6 (DIN): now also U3.2 (DOUT); no longer U3.3 (DOUT)
- net at U1.2 (DOUT): now also U2.6 (DIN); no longer U2.5 (DCKI)
- net at U1.3 (DCKO): now also U2.5 (DCKI); no longer U2.6 (DIN)
- net at U2.2 (DOUT): now also U3.6 (DIN); no longer U3.5 (DCKI)
- net at U2.3 (DCKO): now also U3.5 (DCKI); no longer U3.6 (DIN)
- net at U6.5 (DCKI): now also U5.3 (DCKO); no longer U5.2 (DCKO)
- net at U6.6 (DIN): now also U5.2 (DOUT); no longer U5.3 (DOUT)
