File: kicad/zandvoort_10x10/rgb_led_track_chain.kicad_sch (KiCad schematic)
At the start: 34 parts, among them U10 HD108-2020, U11 HD108-2020, U12 HD108-2020, U13 HD108-2020, U14 HD108-2020, U15 HD108-2020, U16 HD108-2020, U17 HD108-2020, U18 HD108-2020, U19 HD108-2020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

Commit message: Create seaparate 20x20 and 10x10 Kicad projects in kicad root
Connections:
- net CLOCK_CHAIN_1_TO_2: now also U16.3 (DCKO); no longer U16.2 (DCKO)
- net CLOCK_CHAIN_2_TO_3: now also U25.3 (DCKO); no longer U25.2 (DCKO)
- net CLOCK_CHAIN_3_TO_4: now also U34.3 (DCKO); no longer U34.2 (DCKO)
- net DATA_CHAIN_1_TO_2: now also U16.2 (DOUT); no longer U16.3 (DOUT)
- net DATA_CHAIN_2_TO_3: now also U25.2 (DOUT); no longer U25.3 (DOUT)
- net DATA_CHAIN_3_TO_4: now also U34.2 (DOUT); no longer U34.3 (DOUT)
- net DCKO: now also U36.3 (DCKO); no longer U36.2 (DCKO)
- net DOUT: now also U36.2 (DOUT); no longer U36.3 (DOUT)
- net at U34.5 (DCKI): now also U33.3 (DCKO); no longer U33.2 (DCKO)
- net at U34.6 (DIN): now also U33.2 (DOUT); no longer U33.3 (DOUT)
- net at U36.5 (DCKI): now also U35.3 (DCKO); no longer U35.2 (DCKO)
- net at U36.6 (DIN): now also U35.2 (DOUT); no longer U35.3 (DOUT)
- net at U17.2 (DOUT): now also U18.6 (DIN); no longer U18.5 (DCKI)
- net at U17.3 (DCKO): now also U18.5 (DCKI); no longer U18.6 (DIN)
- net at U31.2 (DOUT): now also U32.6 (DIN); no longer U32.5 (DCKI)
- net at U31.3 (DCKO): now also U32.5 (DCKI); no longer U32.6 (DIN)
- net at U31.5 (DCKI): now also U30.3 (DCKO); no longer U30.2 (DCKO)
- net at U31.6 (DIN): now also U30.2 (DOUT); no longer U30.3 (DOUT)
- net at U32.2 (DOUT): now also U33.6 (DIN); no longer U33.5 (DCKI)
- net at U32.3 (DCKO): now also U33.5 (DCKI); no longer U33.6 (DIN)
- net at U11.2 (DOUT): now also U12.6 (DIN); no longer U12.5 (DCKI)
- net at U11.3 (DCKO): now also U12.5 (DCKI); no longer U12.6 (DIN)
- net at U11.5 (DCKI): now also U10.3 (DCKO); no longer U10.2 (DCKO)
- net at U11.6 (DIN): now also U10.2 (DOUT); no longer U10.3 (DOUT)
- net at U22.2 (DOUT): now also U23.6 (DIN); no longer U23.5 (DCKI)
- net at U22.3 (DCKO): now also U23.5 (DCKI); no longer U23.6 (DIN)
- net at U22.5 (DCKI): now also U21.3 (DCKO); no longer U21.2 (DCKO)
- net at U22.6 (DIN): now also U21.2 (DOUT); no longer U21.3 (DOUT)
- net at U25.5 (DCKI): now also U24.3 (DCKO); no longer U24.2 (DCKO)
- net at U25.6 (DIN): now also U24.2 (DOUT); no longer U24.3 (DOUT)
- net at U8.2 (DOUT): now also U9.6 (DIN); no longer U9.5 (DCKI)
- net at U8.3 (DCKO): now also U9.5 (DCKI); no longer U9.6 (DIN)
- net at U8.5 (DCKI): now also U7.3 (DCKO); no longer U7.2 (DCKO)
- net at U8.6 (DIN): now also U7.2 (DOUT); no longer U7.3 (DOUT)
- net at U27.2 (DOUT): now also U28.6 (DIN); no longer U28.5 (DCKI)
- net at U27.3 (DCKO): now also U28.5 (DCKI); no longer U28.6 (DIN)
- net at U27.5 (DCKI): now also U26.3 (DCKO); no longer U26.2 (DCKO)
- net at U27.6 (DIN): now also U26.2 (DOUT); no longer U26.3 (DOUT)
- net at U30.5 (DCKI): now also U29.3 (DCKO); no longer U29.2 (DCKO)
- net at U30.6 (DIN): now also U29.2 (DOUT); no longer U29.3 (DOUT)
- net at U20.2 (DOUT): now also U21.6 (DIN); no longer U21.5 (DCKI)
- net at U20.3 (DCKO): now also U21.5 (DCKI); no longer U21.6 (DIN)
- net at U20.5 (DCKI): now also U19.3 (DCKO); no longer U19.2 (DCKO)
- net at U20.6 (DIN): now also U19.2 (DOUT); no longer U19.3 (DOUT)
- net at U24.5 (DCKI): now also U23.3 (DCKO); no longer U23.2 (DCKO)
- net at U24.6 (DIN): now also U23.2 (DOUT); no longer U23.3 (DOUT)
- net at U16.5 (DCKI): now also U15.3 (DCKO); no longer U15.2 (DCKO)
- net at U16.6 (DIN): now also U15.2 (DOUT); no longer U15.3 (DOUT)
- net at U9.2 (DOUT): now also U10.6 (DIN); no longer U10.5 (DCKI)
- net at U9.3 (DCKO): now also U10.5 (DCKI); no longer U10.6 (DIN)
- net at U14.2 (DOUT): now also U15.6 (DIN); no longer U15.5 (DCKI)
- net at U14.3 (DCKO): now also U15.5 (DCKI); no longer U15.6 (DIN)
- net at U14.5 (DCKI): now also U13.3 (DCKO); no longer U13.2 (DCKO)
- net at U14.6 (DIN): now also U13.2 (DOUT); no longer U13.3 (DOUT)
- net at U13.5 (DCKI): now also U12.3 (DCKO); no longer U12.2 (DCKO)
- net at U13.6 (DIN): now also U12.2 (DOUT); no longer U12.3 (DOUT)
- net at U28.2 (DOUT): now also U29.6 (DIN); no longer U29.5 (DCKI)
- net at U28.3 (DCKO): now also U29.5 (DCKI); no longer U29.6 (DIN)
- net at U18.2 (DOUT): now also U19.6 (DIN); no longer U19.5 (DCKI)
- net at U18.3 (DCKO): now also U19.5 (DCKI); no longer U19.6 (DIN)
