File: kicad/zandvoort_20x20/rgb_led_track_chain.kicad_sch (KiCad schematic)
At the start: 34 parts

Commit message: Add additional LEDs through hierarchical sheets
Parts:
- gave numbers to parts that had none: 34

Commit message: Add leds to schematic and place in layout
Parts:
- renumbered C97 to C100, C98 to C101, C99 to C102, C100 to C103, U97 to U100, U98 to U101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

Commit message: KiCad - Update designator numbers for LEDS
Parts:
- renumbered C103 to C100, C100 to C97, C101 to C98, C102 to C99, U103 to U100, U104 to U101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
